File: ergogen/output/pcbs/Alias.kicad_pcb (KiCad board)
At the start: 2 copper layers, 252.6 x 123.5 mm, 93 parts

Commit message: update case compatibility
Other:
- net class Default added: clearance 0.2, trace_width 0.25, via_dia 0.8, via_drill 0.4

Commit message: update readme
Other:
- board size 252.6 x 123.5 mm -> 254 x 125.2 mm
