File: ergogen/output/pcbs/case_bottom.kicad_pcb (KiCad board)
At the start: 2 copper layers, 252.6 x 123.5 mm, 36 parts

Commit message: update case compatibility
Other:
- outline, holes or cut-outs redrawn

Commit message: update readme
Other:
- board size 252.6 x 123.5 mm -> 254 x 125.2 mm
